Commit message: Update launch, URDF, EKF config, and new pose calculator script

File: urdf/robot.urdf.xacro (robot description, xacro)
@@ -39,5 +39,5 @@
     <parent link="base_link"/>
     <child link="imu_link"/>
-    <origin xyz="0.0 0.0 0.06" rpy="0 3.141592653589793 0"/>
+    <origin xyz="0.0 0.0 0.06" rpy="0 0 0"/>
   </joint>
   <!-- ========================================= -->
@@ -64,5 +64,5 @@
     Reversed values:
     -->
-    <origin xyz="0.045 0.0575 0.0" rpy="-1.5708 0 -1.5708"/>
+    <origin xyz="0.045 0 0.0" rpy="1.5708 0 1.5708"/>
   </joint>
 </robot>
