Commit message: Updated EKF config, launch file, and added alternate URDF

File: urdf/robot.urdf2.xacro (robot description, xacro)
@@ -39,5 +39,5 @@
     <parent link="base_link"/>
     <child link="imu_link"/>
-    <origin xyz="0.0 0.0 0.18" rpy="0 0 0"/>
+    <origin xyz="0.0 0.0 0.18" rpy="3.141592 0 0"/>
   </joint>
   <!-- ========================================= -->
